File: hardware/putikeeg_cw_trainer.kicad_sch (KiCad schematic)
At the start: 54 parts, among them J1 Prog, J2 128x64 LCD, J3 Battery, J4 KEY, J5 PH, J6 LCD Backlight, J7 POT_A, J8 POT_B, P1 USB_C_Plug_USB2.0, Q2 SS8050, Q3 SS8550, Q4 SS8550, Q5 IRFR9020TRPBF-HXY, Q6 SS8050, SW1 SW_Menu, SW2 SW_Prev, SW3 SW_Next, SW4 SW_Enter, SW5 SW_Pwr, U1 STC8H3K64S2-LQFP32, U2 TP4056-42-ESOP8, U3 HT7833, U4 HX4004A

Commit message: Drive the LCD backlight active high with the P0.3 pull-up
The corrected schematic shows that P0.3 drives the Q6 base through a
120 ohm resistor, with a 47 kohm pull-down, so a high pin turns the
backlight on. The pin runs open drain with the internal pull-up,
because a push-pull high would source over 20 mA into the base.
Parts:
- R10: value R -> 47k
- R2: value R -> 120
Connections:
- net GND: now also Q6.2 (E), R10.2
- net P0.3: now also R10.1, R2.1; no longer R10.2
- net VCC: no longer R2.1
Other:
- moved on the sheet: R10
Changed lines of the file:
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@@
 	)
 	(junction
+		(at 21.59 104.14)
+		(diameter 0)
+		(color 0 0 0 0)
+	)
+	(junction
 		(at 234.95 144.78)
 		(diameter 0)
@@
 	(wire
 		(pts
+			(xy 39.37 109.22) (xy 39.37 111.76)
+		)
+		(stroke
+			(width 0)
+			(type default)
+		)
+	)
+	(wire
+		(pts
 			(xy 242.57 80.01) (xy 242.57 81.28)
 		)
@@
 	(wire
 		(pts
-			(xy 166.37 181.61) (xy 158.75 181.61)
+			(xy 16.51 104.14) (xy 21.59 104.14)
 		)
 		(stroke
@@
 	(wire
 		(pts
-			(xy 199.39 114.3) (xy 212.09 114.3)
+			(xy 166.37 181.61) (xy 158.75 181.61)
 		)
 		(stroke
@@
 	(wire
 		(pts
-			(xy 55.88 123.19) (xy 55.88 124.46)
+			(xy 199.39 114.3) (xy 212.09 114.3)
 		)
 		(stroke
@@
 	(wire
 		(pts
-			(xy 21.59 102.87) (xy 21.59 104.14)
+			(xy 55.88 123.19) (xy 55.88 124.46)
 		)
 		(stroke
@@
 	(wire
 		(pts
+			(xy 21.59 104.14) (xy 21.59 106.68)
+		)
+		(stroke
+			(width 0)
+			(type default)
+		)
+	)
+	(wire
+		(pts
 			(xy 233.68 128.27) (xy 237.49 128.27)
 		)
@@
 	(wire
 		(pts
-			(xy 39.37 109.22) (xy 39.37 110.49)
-		)
-		(stroke
-			(width 0)
-			(type default)
-		)
-	)
-	(wire
-		(pts
 			(xy 171.45 35.56) (xy 171.45 34.29)
 		)
@@
 	(wire
 		(pts
-			(xy 39.37 118.11) (xy 39.37 123.19)
-		)
-		(stroke
-			(width 0)
-			(type default)
-		)
-	)
-	(wire
-		(pts
 			(xy 160.02 97.79) (xy 160.02 99.06)
 		)
@@
 	)
 	(label "P0.3"
-		(at 39.37 123.19 90)
+		(at 16.51 104.14 0)
 		(effects
 			(font
@@
 	)
 	(symbol
-		(lib_id "power:VCC")
-		(at 21.59 102.87 0)
-		(unit 1)
-		(body_style 1)
-		(exclude_from_sim no)
-		(in_bom yes)
-		(on_board yes)
-		(in_pos_files yes)
-		(dnp no)
-		(fields_autoplaced yes)
-		(property "Reference" "#PWR026"
-			(at 21.59 106.68 0)
-			(hide yes)
-			(show_name no)
-			(do_not_autoplace no)
-			(effects
-				(font
-					(size 1.27 1.27)
-				)
-			)
-		)
-		(property "Value" "VCC"
-			(at 21.59 97.79 0)
-			(show_name no)
-			(do_not_autoplace no)
-			(effects
-				(font
-					(size 1.27 1.27)
-				)
-			)
-		)
-		(property "Footprint" ""
-			(at 21.59 102.87 0)
-			(hide yes)
-			(show_name no)
-			(do_not_autoplace no)
-			(effects
-				(font
-					(size 1.27 1.27)
-				)
-			)
-		)
-		(property "Datasheet" ""
-			(at 21.59 102.87 0)
-			(hide yes)
-			(show_name no)
-			(do_not_autoplace no)
-			(effects
-				(font
-					(size 1.27 1.27)
-				)
-			)
-		)
-		(property "Description" "Power symbol creates a global label with name \"VCC\""
-			(at 21.59 102.87 0)
-			(hide yes)
-			(show_name no)
-			(do_not_autoplace no)
-			(effects
-				(font
-					(size 1.27 1.27)
-				)
-			)
-		)
-		(pin "1"
-		)
-		(instances
-			(project "putikeeg_cw_trainer"
-				(path "/a64e981c-da55-4356-9f6e-aef3e7ccd7d2"
-					(reference "#PWR026")
-					(unit 1)
-				)
-			)
-		)
-	)
-	(symbol
 		(lib_id "Switch:SW_Push_Dual")
 		(at 229.87 29.21 0)
@@
 	)
 	(symbol
+		(lib_id "power:GND")
+		(at 39.37 111.76 0)
+		(unit 1)
+		(body_style 1)
+		(exclude_from_sim no)
+		(in_bom yes)
+		(on_board yes)
+		(in_pos_files yes)
+		(dnp no)
+		(fields_autoplaced yes)
+		(property "Reference" "#PWR043"
+			(at 39.37 118.11 0)
+			(hide yes)
+			(show_name no)
+			(do_not_autoplace no)
+			(effects
+				(font
+					(size 1.27 1.27)
+				)
+			)
+		)
+		(property "Value" "GND"
+			(at 39.37 116.84 0)
+			(show_name no)
+			(do_not_autoplace no)
+			(effects
+				(font
+					(size 1.27 1.27)
+				)
+			)
+		)
+		(property "Footprint" ""
+			(at 39.37 111.76 0)
+			(hide yes)
+			(show_name no)
+			(do_not_autoplace no)
+			(effects
+				(font
+					(size 1.27 1.27)
+				)
+			)
+		)
+		(property "Datasheet" ""
+			(at 39.37 111.76 0)
+			(hide yes)
+			(show_name no)
+			(do_not_autoplace no)
+			(effects
+				(font
+					(size 1.27 1.27)
+				)
+			)
+		)
+		(property "Description" "Power symbol creates a global label with name \"GND\" , ground"
+			(at 39.37 111.76 0)
+			(hide yes)
+			(show_name no)
+			(do_not_autoplace no)
+			(effects
+				(font
+					(size 1.27 1.27)
+				)
+			)
+		)
+		(pin "1"
+		)
+		(instances
+			(project "putikeeg_cw_trainer"
+				(path "/a64e981c-da55-4356-9f6e-aef3e7ccd7d2"
+					(reference "#PWR043")
+					(unit 1)
+				)
+			)
+		)
+	)
+	(symbol
 		(lib_id "Local:HX4004A-SOT-23-6")
 		(at 222.25 118.11 0)
@@
 			)
 		)
-		(property "Value" "R"
+		(property "Value" "120"
 			(at 26.67 100.33 90)
 			(show_name no)
@@
 	)
 	(symbol
+		(lib_id "power:GND")
+		(at 21.59 114.3 0)
+		(unit 1)
+		(body_style 1)
+		(exclude_from_sim no)
+		(in_bom yes)
+		(on_board yes)
+		(in_pos_files yes)
+		(dnp no)
+		(fields_autoplaced yes)
+		(property "Reference" "#PWR042"
+			(at 21.59 120.65 0)
+			(hide yes)
+			(show_name no)
+			(do_not_autoplace no)
+			(effects
+				(font
+					(size 1.27 1.27)
+				)
+			)
+		)
+		(property "Value" "GND"
+			(at 21.59 119.38 0)
+			(show_name no)
+			(do_not_autoplace no)
+			(effects
+				(font
+					(size 1.27 1.27)
+				)
+			)
+		)
+		(property "Footprint" ""
+			(at 21.59 114.3 0)
+			(hide yes)
+			(show_name no)
+			(do_not_autoplace no)
+			(effects
+				(font
+					(size 1.27 1.27)
+				)
+			)
+		)
+		(property "Datasheet" ""
+			(at 21.59 114.3 0)
+			(hide yes)
+			(show_name no)
+			(do_not_autoplace no)
+			(effects
+				(font
+					(size 1.27 1.27)
+				)
+			)
+		)
+		(property "Description" "Power symbol creates a global label with name \"GND\" , ground"
+			(at 21.59 114.3 0)
+			(hide yes)
+			(show_name no)
+			(do_not_autoplace no)
+			(effects
+				(font
+					(size 1.27 1.27)
+				)
+			)
+		)
+		(pin "1"
+		)
+		(instances
+			(project "putikeeg_cw_trainer"
+				(path "/a64e981c-da55-4356-9f6e-aef3e7ccd7d2"
+					(reference "#PWR042")
+					(unit 1)
+				)
+			)
+		)
+	)
+	(symbol
 		(lib_id "Device:R")
-		(at 39.37 114.3 0)
+		(at 21.59 110.49 0)
 		(unit 1)
 		(body_style 1)
@@
 		(fields_autoplaced yes)
 		(property "Reference" "R10"
-			(at 41.91 113.0299 0)
+			(at 24.13 109.2199 0)
 			(show_name no)
 			(do_not_autoplace no)
@@
 			)
 		)
-		(property "Value" "R"
-			(at 41.91 115.5699 0)
+		(property "Value" "47k"
+			(at 24.13 111.7599 0)
 			(show_name no)
 			(do_not_autoplace no)
@@
 		)
 		(property "Footprint" ""
-			(at 37.592 114.3 90)
+			(at 19.812 110.49 90)
 			(hide yes)
 			(show_name no)
@@
 		)
 		(property "Datasheet" ""
-			(at 39.37 114.3 0)
+			(at 21.59 110.49 0)
 			(hide yes)
 			(show_name no)
@@
 		)
 		(property "Description" "Resistor"
-			(at 39.37 114.3 0)
+			(at 21.59 110.49 0)
 			(hide yes)
 			(show_name no)
